Commit message: add friction for TPU socks

File: sim/optimus_primal.urdf (robot description, URDF)
Before this commit: robot optimus_primal, 9 links, 8 joints
Links:
- added link foot_fl, mass 0.005; collision sphere radius=0.012; visual sphere radius=0.012
- added link foot_fr, mass 0.005; collision sphere radius=0.012; visual sphere radius=0.012
- added link foot_rl, mass 0.005; collision sphere radius=0.012; visual sphere radius=0.012
- added link foot_rr, mass 0.005; collision sphere radius=0.012; visual sphere radius=0.012
Joints:
- added joint foot_joint_fl: type fixed, parent lower_link_fl, child foot_fl, origin xyz=0 0 -0.104 rpy=0 0 0
- added joint foot_joint_fr: type fixed, parent lower_link_fr, child foot_fr, origin xyz=0 0 -0.104 rpy=0 0 0
- added joint foot_joint_rl: type fixed, parent lower_link_rl, child foot_rl, origin xyz=0 0 -0.104 rpy=0 0 0
- added joint foot_joint_rr: type fixed, parent lower_link_rr, child foot_rr, origin xyz=0 0 -0.104 rpy=0 0 0

Commit message: 1.292kg mass model, interp+tilt+sigma sweep, rank_gaits

File: sim/optimus_primal.urdf (robot description, URDF)
Before this commit: robot optimus_primal, 13 links, 12 joints
Links:
- link base_link: mass 0.6 -> 0.672
- link lower_link_fl: mass 0.04 -> 0.065
- link lower_link_fr: mass 0.04 -> 0.065
- link lower_link_rl: mass 0.04 -> 0.065
- link lower_link_rr: mass 0.04 -> 0.065
- link upper_link_fl: mass 0.06 -> 0.085
- link upper_link_fr: mass 0.06 -> 0.085
- link upper_link_rl: mass 0.06 -> 0.085
- link upper_link_rr: mass 0.06 -> 0.085
